File: pcb/indoor-bme280.sch (KiCad schematic (older format))
At the start: 14 parts, among them IC1 ATMEGA328P-A, P1 SOLAR, P2 CAP, P3 CONN_02X03, P4 BME280, P5 ANT

Commit message: updated kicad
Parts:
- P3: value CONN_02X03 -> ISP
Connections:
- no-connect marks 11 -> 23
Changed lines of the file:
@@
 LIBS:valves
 LIBS:rfm69
+LIBS:indoor-bme280-cache
 EELAYER 25 0
 EELAYER END
@@
 P 5350 2050
 F 0 "P3" H 5350 2250 50  0000 C CNN
-F 1 "CONN_02X03" H 5350 1850 50  0000 C CNN
+F 1 "ISP" H 5350 1850 50  0000 C CNN
 F 2 "Pin_Headers:Pin_Header_Straight_2x03" H 5350 850 50  0001 C CNN
 F 3 "" H 5350 850 50  0000 C CNN
@@
 Wire Wire Line
 	3350 4200 3650 4200
+NoConn ~ 3350 2850
+NoConn ~ 3350 2950
+NoConn ~ 3350 3450
+NoConn ~ 3350 3550
+NoConn ~ 3350 3700
+NoConn ~ 3350 3800
+NoConn ~ 3350 3900
+NoConn ~ 3350 4000
+NoConn ~ 3350 4850
+NoConn ~ 3350 4950
+NoConn ~ 3350 5050
+NoConn ~ 3350 5150
 $EndSCHEMATC
