File: pcb/indoor-temperature-sensor/indoor-temperature-sensor.sch (KiCad schematic (older format))
At the start: 30 parts, among them IC1 TP4056, J1 BATT, J2 USB, J3 PROG, J4 ePaper, J5 BME280, J6 TOUCH, Q1 BC327, Q2 BC337, SW1 RST, U1 ESP32-WROOM-32D

Commit message: wip
Parts:
- removed J1: BATT, symbol Connector:Conn_01x03_Male
- added C3, C8, C9: 10uF, Capacitor_SMD:C_0805_2012Metric, symbol Device:C
- added C5: 100nF, Capacitor_SMD:C_0805_2012Metric, symbol Device:C
- added J2: BATT, Connector_PinHeader_2.00mm:PinHeader_1x02_P2.00mm_Vertical, symbol Connector:Conn_01x02_Male
- added J4: PW, Connector_PinHeader_2.54mm:PinHeader_1x03_P2.54mm_Vertical, symbol Connector:Conn_01x03_Male
- added L1: 1.5uH Murata, coil:Murata 1266AS-H-1R5N=P2, symbol Device:L
- added U1: TPS63031DSKT, tps6303x:VSON-10-1EP_2.x2.5mm_P0.5mm_EP1.2x2mm, symbol tps63031dskt:TPS63031DSKT
- C1, C2: footprint (none) -> Capacitor_SMD:C_0805_2012Metric
- C10: renamed from C6; footprint (none) -> Capacitor_SMD:C_0805_2012Metric
- C4: renamed from C3; footprint (none) -> Capacitor_SMD:C_0805_2012Metric
- C6: renamed from C4; footprint (none) -> Capacitor_Tantalum_SMD:CP_EIA-7343-43_Kemet-X_Pad2.25x2.55mm_HandSolder
- C7: renamed from C5; footprint (none) -> Capacitor_SMD:C_0805_2012Metric
- D1: footprint (none) -> Diode_THT:D_A-405_P2.54mm_Vertical_AnodeUp
- IC1: footprint (none) -> Package_SO:SOIC-8_3.9x4.9mm_P1.27mm
- J1: renamed from J2; footprint (none) -> Connector_PinHeader_2.00mm:PinHeader_1x02_P2.00mm_Vertical
- J3: footprint (none) -> Connector_PinHeader_2.54mm:PinHeader_2x03_P2.54mm_Vertical
- J5: renamed from J4; footprint (none) -> Connector_PinHeader_2.00mm:PinHeader_1x08_P2.00mm_Vertical
- J6: renamed from J5; footprint (none) -> Connector_PinHeader_2.54mm:PinHeader_1x04_P2.54mm_Vertical
- J7: renamed from J6; footprint (none) -> Connector_PinHeader_1.00mm:PinHeader_1x01_P1.00mm_Vertical
- Q1, Q2: footprint Package_TO_SOT_THT:TO-92_Inline -> Package_TO_SOT_THT:TO-92
- R1, R10, R11, R12, R2, R3, R4, R5, R6, R7, R8, R9: footprint (none) -> Resistor_SMD:R_0805_2012Metric
- SW1: footprint (none) -> Connector_PinHeader_2.54mm:PinHeader_1x02_P2.54mm_Vertical
- renumbered U1 to U2
Connections:
- net +3V3: now also J4.2 (Pin_2)
- net +BATT: now also C3.1, J2.1 (Pin_1), U1.5 (VIN)
- net GND: now also C3.2, C5.1, C8.2, C9.2, J2.2 (Pin_2), J4.1 (Pin_1), U1.3 (PGND), U1.9 (GND)
- new net: C8.1, C9.1, J4.3 (Pin_3), U1.1 (VOUT), U1.10 (FB)
- new net: C5.2, U1.6 (EN), U1.7 (PS/SYNC), U1.8 (VINA)
- new net: L1.1, U1.4 (L1)
- new net: L1.2, U1.2 (L2)
Other:
- moved on the sheet: R3, R4
