File: pcb/buck-boost-33/buck-boost-33.sch (KiCad schematic (older format))
At the start: 14 parts, among them IC1 TP4056, J1 BATT, J2 buck-boost-conn, J3 PWR, U1 TPS63031DSKT

Commit message: rework with new footprints
Parts:
- L1: footprint coil:Murata 1266AS-H-1R5N=P2 -> coil:Murata_1266AS-H-1R5N=P2
Connections:
- net labels added: 3.3V
- wire segments 58 -> 59
Changed lines of the file:
@@
 F 0 "L1" V 4840 4100 50  0000 C CNN
 F 1 "L" V 4749 4100 50  0000 C CNN
-F 2 "coil:Murata 1266AS-H-1R5N=P2" H 4650 4100 50  0001 C CNN
+F 2 "coil:Murata_1266AS-H-1R5N=P2" H 4650 4100 50  0001 C CNN
 F 3 "~" H 4650 4100 50  0001 C CNN
 	1    4650 4100
@@
 L power:GND #PWR08
 U 1 1 5EF948DE
-P 5100 4850
-F 0 "#PWR08" H 5100 4600 50  0001 C CNN
-F 1 "GND" H 5105 4677 50  0000 C CNN
-F 2 "" H 5100 4850 50  0001 C CNN
-F 3 "" H 5100 4850 50  0001 C CNN
-	1    5100 4850
+P 5100 5800
+F 0 "#PWR08" H 5100 5550 50  0001 C CNN
+F 1 "GND" H 5105 5627 50  0000 C CNN
+F 2 "" H 5100 5800 50  0001 C CNN
+F 3 "" H 5100 5800 50  0001 C CNN
+	1    5100 5800
 	1    0    0    -1
 $EndComp
@@
 Wire Wire Line
 	4700 4250 5100 4250
-Wire Wire Line
-	5100 4250 5100 4850
 Wire Wire Line
 	5700 4850 6150 4850
@@
 Wire Wire Line
 	6450 4650 6450 3700
-Wire Wire Line
-	6450 3700 7750 3700
-Wire Wire Line
-	7750 3700 7750 4350
-Text GLabel 7600 4150 1    50   Input ~ 0
+Text GLabel 7700 4150 1    50   Input ~ 0
 BATT
-Wire Wire Line
-	7600 4150 7600 4350
 Text GLabel 7100 4750 0    50   Input ~ 0
 CHRG
@@
 Wire Wire Line
 	2200 3900 2500 3900
+Wire Wire Line
+	5100 4250 5100 5800
+Wire Wire Line
+	7850 3700 7850 4350
+Wire Wire Line
+	6450 3700 7850 3700
+Wire Wire Line
+	7700 4150 7700 4350
+$Comp
+L power:+5V #PWR0101
+U 1 1 5EFE9906
+P 7550 4150
+F 0 "#PWR0101" H 7550 4000 50  0001 C CNN
+F 1 "+5V" H 7565 4323 50  0000 C CNN
+F 2 "" H 7550 4150 50  0001 C CNN
+F 3 "" H 7550 4150 50  0001 C CNN
+	1    7550 4150
+	1    0    0    -1
+$EndComp
+Wire Wire Line
+	7550 4150 7550 4350
+Text Label 7750 3700 0    50   ~ 0
+3.3V
 $EndSCHEMATC

Commit message: add LCSC part numbers, use another coil
Parts:
- C1, C2, C4, C5, C6: LCSC (none) -> C100083
- C3: LCSC (none) -> C386062
- IC1: LCSC (none) -> C16581
- L1: footprint coil:Murata_1266AS-H-1R5N=P2 -> coil:CoilMX-MS0420; LCSC (none) -> C380153
- R1: LCSC (none) -> C253349
- R2: LCSC (none) -> C17661
- U1: LCSC (none) -> C15516
Changed lines of the file:
@@
 F 2 "tps6303x:VSON-10-1EP_2.x2.5mm_P0.5mm_EP1.2x2mm" H 4450 4550 50  0001 C CNN
 F 3 "http://www.ti.com/lit/ds/symlink/tps63031.pdf?HQS=TI-null-null-mousermode-df-pf-null-wwe&ts=1591517168701&ref_url=https://www.mouser.de/" H 4450 4550 50  0001 C CNN
+F 4 "C15516" H 4450 4550 50  0001 C CNN "LCSC"
 	1    4450 4550
 	0    1    1    0
@@
 F 2 "Capacitor_SMD:C_0805_2012Metric" H 4700 6150 50  0001 C CNN
 F 3 "~" H 4700 6150 50  0001 C CNN
+F 4 "C386062" H 4700 6150 50  0001 C CNN "LCSC"
 	1    4700 6150
 	-1   0    0    1
@@
 F 2 "Capacitor_SMD:C_0805_2012Metric" H 5700 4750 50  0001 C CNN
 F 3 "~" H 5700 4750 50  0001 C CNN
+F 4 "C100083" H 5700 4750 50  0001 C CNN "LCSC"
 	1    5700 4750
 	-1   0    0    1
@@
 F 2 "Capacitor_SMD:C_0805_2012Metric" H 6150 4750 50  0001 C CNN
 F 3 "~" H 6150 4750 50  0001 C CNN
+F 4 "C100083" H 6150 4750 50  0001 C CNN "LCSC"
 	1    6150 4750
 	-1   0    0    1
@@
 F 2 "Capacitor_SMD:C_0805_2012Metric" H 3900 4750 50  0001 C CNN
 F 3 "~" H 3900 4750 50  0001 C CNN
+F 4 "C100083" H 3900 4750 50  0001 C CNN "LCSC"
 	1    3900 4750
 	-1   0    0    1
@@
 F 0 "L1" V 4840 4100 50  0000 C CNN
 F 1 "L" V 4749 4100 50  0000 C CNN
-F 2 "coil:Murata_1266AS-H-1R5N=P2" H 4650 4100 50  0001 C CNN
+F 2 "coil:CoilMX-MS0420" H 4650 4100 50  0001 C CNN
 F 3 "~" H 4650 4100 50  0001 C CNN
+F 4 "C380153" V 4650 4100 50  0001 C CNN "LCSC"
 	1    4650 4100
 	0    -1   -1   0
@@
 F 2 "Package_SO:SOIC-8_3.9x4.9mm_P1.27mm" H 4400 2500 50  0001 C CNN
 F 3 "" H 4650 2600 50  0001 C CNN
+F 4 "C16581" H 4650 2600 50  0001 C CNN "LCSC"
 	1    4650 2600
 	1    0    0    -1
@@
 F 2 "Resistor_SMD:R_0805_2012Metric" V 5180 2550 50  0001 C CNN
 F 3 "~" H 5250 2550 50  0001 C CNN
+F 4 "C17661" H 5250 2550 50  0001 C CNN "LCSC"
 	1    5250 2550
 	1    0    0    -1
@@
 F 2 "Capacitor_SMD:C_0805_2012Metric" H 6000 2100 50  0001 C CNN
 F 3 "~" H 6000 2100 50  0001 C CNN
+F 4 "C100083" H 6000 2100 50  0001 C CNN "LCSC"
 	1    6000 2100
 	1    0    0    -1
@@
 F 2 "Capacitor_SMD:C_0805_2012Metric" H 3750 1950 50  0001 C CNN
 F 3 "~" H 3750 1950 50  0001 C CNN
+F 4 "C100083" H 3750 1950 50  0001 C CNN "LCSC"
 	1    3750 1950
 	1    0    0    -1
@@
 F 2 "Resistor_SMD:R_0805_2012Metric" V 3680 1600 50  0001 C CNN
 F 3 "~" H 3750 1600 50  0001 C CNN
+F 4 "C253349" H 3750 1600 50  0001 C CNN "LCSC"
 	1    3750 1600
 	1    0    0    -1

Commit message: back to marata inductor; smaller pcb
Parts:
- L1: footprint coil:CoilMX-MS0420 -> coil:Murata_1266AS-H-1R5N=P2; LCSC C380153 -> (none)
Changed lines of the file:
@@
 F 0 "L1" V 4840 4100 50  0000 C CNN
 F 1 "L" V 4749 4100 50  0000 C CNN
-F 2 "coil:CoilMX-MS0420" H 4650 4100 50  0001 C CNN
+F 2 "coil:Murata_1266AS-H-1R5N=P2" H 4650 4100 50  0001 C CNN
 F 3 "~" H 4650 4100 50  0001 C CNN
-F 4 "C380153" V 4650 4100 50  0001 C CNN "LCSC"
 	1    4650 4100
 	0    -1   -1   0

Commit message: update
Parts:
- added R3, R4: 0, Resistor_SMD:R_0805_2012Metric, symbol Device:R
Connections:
- net BATT: now also U1.6 (EN), R4.2
- net GND: now also R3.2
- net at C3.2, U1.8 (VINA): no longer U1.6 (EN), U1.7 (PS/SYNC)
- new net: R3.1, R4.1, U1.7 (PS/SYNC)
Changed lines of the file:
@@
 	4500 4200 4500 4100
 Wire Wire Line
-	4500 4500 3900 4500
+	4500 4500 4200 4500
 Wire Wire Line
 	3900 4500 3900 4650
@@
 Wire Wire Line
 	4700 6250 4700 6350
-Wire Wire Line
-	4700 5300 4600 5300
-Connection ~ 4700 5300
-Wire Wire Line
-	4600 5300 4500 5300
-Connection ~ 4600 5300
 Wire Wire Line
 	5700 4650 6150 4650
@@
 Text Label 7750 3700 0    50   ~ 0
 3.3V
+Wire Wire Line
+	4200 4500 4200 5300
+Wire Wire Line
+	4200 5300 4500 5300
+Connection ~ 4200 4500
+Wire Wire Line
+	4200 4500 4000 4500
+$Comp
+L Device:R R3
+U 1 1 5F008EF1
+P 4300 5650
+F 0 "R3" H 4370 5696 50  0000 L CNN
+F 1 "0" H 4370 5605 50  0000 L CNN
+F 2 "Resistor_SMD:R_0805_2012Metric" V 4230 5650 50  0001 C CNN
+F 3 "~" H 4300 5650 50  0001 C CNN
+	1    4300 5650
+	1    0    0    -1
+$EndComp
+$Comp
+L power:GND #PWR016
+U 1 1 5F00B59A
+P 4300 5850
+F 0 "#PWR016" H 4300 5600 50  0001 C CNN
+F 1 "GND" H 4305 5677 50  0000 C CNN
+F 2 "" H 4300 5850 50  0001 C CNN
+F 3 "" H 4300 5850 50  0001 C CNN
+	1    4300 5850
+	1    0    0    -1
+$EndComp
+Wire Wire Line
+	4600 5300 4600 5500
+Wire Wire Line
+	4600 5500 4300 5500
+Wire Wire Line
+	4300 5800 4300 5850
+$Comp
+L Device:R R4
+U 1 1 5F00EEC8
+P 4050 5650
+F 0 "R4" H 4120 5696 50  0000 L CNN
+F 1 "0" H 4120 5605 50  0000 L CNN
+F 2 "Resistor_SMD:R_0805_2012Metric" V 3980 5650 50  0001 C CNN
+F 3 "~" H 4050 5650 50  0001 C CNN
+	1    4050 5650
+	1    0    0    -1
+$EndComp
+Wire Wire Line
+	4300 5500 4050 5500
+Connection ~ 4300 5500
+Wire Wire Line
+	4000 4500 4000 5900
+Wire Wire Line
+	4000 5900 4050 5900
+Wire Wire Line
+	4050 5900 4050 5800
+Connection ~ 4000 4500
+Wire Wire Line
+	4000 4500 3900 4500
 $EndSCHEMATC
